Commit message: Adding cartesian controller forward kine

File: robot_description/model/robot.urdf.xacro (robot description, xacro)
@@ -161,15 +161,15 @@
   <link name="endeffector">
     <collision>
-      <origin xyz="0 0 0.057" rpy="0 0 0"/>
+      <origin xyz="0 0 0" rpy="0 0 0"/>
       <geometry>
-        <!--mesh filename="package://niki_arm_description/meshes/base_link2.stl" scale="0.01 0.01 0.01"/ -->
-        <box size="0.05 0.026 0.114"/>
+        <mesh filename="package://robot_description/meshes/endeffector.stl" scale="0.001 0.001 0.001"/>
+        <!--<box size="0.05 0.026 0.076"/>-->
       </geometry>
     </collision>
     <visual>
-      <origin xyz="0 0 0.057" rpy="0 0 0"/>
+      <origin xyz="0 0 0.0" rpy="0 0 0"/>
       <geometry>
-        <!-- <mesh filename="package://niki_arm_description/meshes/base_link2.stl" scale="0.01 0.01 0.01"/> -->
-        <box size="0.05 0.026 0.114"/>
+        <mesh filename="package://robot_description/meshes/endeffector.stl" scale="0.001 0.001 0.001"/>
+        <!--<box size="0.031 0.05 0.076"/>-->
       </geometry>
       <material name="white"/>

Commit message: Adding new stl files with new origin and a dummy grinder

File: robot_description/model/robot.urdf.xacro (robot description, xacro)
@@ -19,15 +19,15 @@
     </inertial>
     <collision>
-      <origin xyz="0 0 0.073" rpy="0 0 0"/>
-      <geometry>
-        <!--mesh filename="package://niki_arm_description/meshes/base_link2.stl" scale="0.01 0.01 0.01"/ -->
-        <box size="0.146 0.146 0.129"/>
-      </geometry>
-    </collision>
-    <visual>
-      <origin xyz="0 0 0.073" rpy="0 0 0"/>
-      <geometry>
-        <!-- <mesh filename="package://niki_arm_description/meshes/base_link2.stl" scale="0.01 0.01 0.01"/> -->
-        <box size="0.146 0.146 0.129"/>
+      <origin xyz="0 0 0.008" rpy="0 0 0"/>
+      <geometry>
+        <mesh filename="package://robot_description/new_meshes/base.stl" scale="0.001 0.001 0.001"/>
+        <!--box size="0.146 0.146 0.129"/ -->
+      </geometry>
+    </collision>
+    <visual>
+      <origin xyz="0 0 0.008" rpy="0 0 0"/>
+      <geometry>
+        <mesh filename="package://robot_description/new_meshes/base.stl" scale="0.001 0.001 0.001"/>
+        <!--box size="0.146 0.146 0.129"/ -->
       </geometry>
       <material name="white"/>
@@ -50,14 +50,14 @@
     </inertial>
 		<visual>
-			<origin xyz="0 0 0.0205" rpy="0 0 0"/>
+			<origin xyz="0 0 0.0" rpy="0 0 0"/>
 			<geometry>
-				<mesh filename="package://robot_description/meshes/mx-64base.stl" scale="0.01 0.01 0.01"/>
+				<mesh filename="package://robot_description/new_meshes/mx-64tobase.stl" scale="0.01 0.01 0.01"/>
 			</geometry>
 			<material name="blue"/>
 		</visual>
 		<collision>
-			<origin xyz="0 0 0.0205" rpy="0 0 0"/>
+			<origin xyz="0 0 0.0" rpy="0 0 0"/>
 			<geometry>
-				<mesh filename="package://robot_description/meshes/mx-64base.stl" scale="0.01 0.01 0.01"/>
+				<mesh filename="package://robot_description/new_meshes/mx-64tobase.stl" scale="0.01 0.01 0.01"/>
 			</geometry>
 		</collision>
@@ -67,5 +67,5 @@
     <parent link="link_1"/>
     <child link="link_2"/>
-    <origin xyz="0 0.0 0.054" rpy="0 0 0"/>
+    <origin xyz="0 0.0 0.044" rpy="0 0 0"/>
     <axis xyz="0 0 1"/>
     <limit velocity="4.8" effort="1" lower="-1.56" upper="1.56" />
@@ -79,14 +79,14 @@
     </inertial>
     <visual>
-      <origin xyz="0 0 0.048" rpy="0 0 0"/>
-      <geometry>
-        <mesh filename="package://robot_description/meshes/mx-64t2.stl" scale="0.01 0.01 0.01"/>
+      <origin xyz="0 0 0.0" rpy="0 0 0"/>
+      <geometry>
+        <mesh filename="package://robot_description/new_meshes/mx-64second.stl" scale="0.01 0.01 0.01"/>
       </geometry>
       <material name="red"/>
     </visual>
     <collision>
-      <origin xyz="0 0 0.048" rpy="0 0 0"/>
-      <geometry>
-        <mesh filename="package://robot_description/meshes/mx-64t2.stl" scale="0.01 0.01 0.01"/>
+      <origin xyz="0 0 0.0" rpy="0 0 0"/>
+      <geometry>
+        <mesh filename="package://robot_description/new_meshes/mx-64second.stl" scale="0.01 0.01 0.01"/>
       </geometry>
     </collision>
@@ -96,5 +96,5 @@
     <parent link="link_2"/>
     <child link="link_3"/>
-    <origin xyz="0 0.0 0.048" rpy="0 0 0"/>
+    <origin xyz="0 0.0 0.058" rpy="0 0 0"/>
     <axis xyz="0 1 0"/>
     <limit velocity="4.8" effort="1" lower="-1.56" upper="1.56" />
@@ -161,15 +161,13 @@
   <link name="endeffector">
     <collision>
-      <origin xyz="0 0 0" rpy="0 0 0"/>
-      <geometry>
-        <mesh filename="package://robot_description/meshes/endeffector.stl" scale="0.001 0.001 0.001"/>
-        <!--<box size="0.05 0.026 0.076"/>-->
-      </geometry>
-    </collision>
-    <visual>
-      <origin xyz="0 0 0.0" rpy="0 0 0"/>
-      <geometry>
-        <mesh filename="package://robot_description/meshes/endeffector.stl" scale="0.001 0.001 0.001"/>
-        <!--<box size="0.031 0.05 0.076"/>-->
+      <origin xyz="0 0 0.0" rpy="0 0 0"/>
+      <geometry>
+        <mesh filename="package://robot_description/new_meshes/endeffector.stl" scale="0.001 0.001 0.001"/>
+      </geometry>
+    </collision>
+    <visual>
+      <origin xyz="0 0 0.0" rpy="0 0 0"/>
+      <geometry>
+        <mesh filename="package://robot_description/new_meshes/endeffector.stl" scale="0.001 0.001 0.001"/>
       </geometry>
       <material name="white"/>
@@ -181,3 +179,30 @@
     </inertial>
   </link>
+  <!-- joint5 -->
+  <joint name="joint5" type="fixed">
+    <parent link="endeffector"/>
+    <child link="link_grinder"/>
+    <origin xyz="0 0 0.065" rpy="0 0 0"/>
+    <axis xyz="0 0 1"/>
+  </joint>
+  <link name="link_grinder">
+    <collision>
+      <origin xyz="0 0 0.0" rpy="0 0 0"/>
+      <geometry>
+        <mesh filename="package://robot_description/new_meshes/grinder.stl" scale="0.001 0.001 0.001"/>
+      </geometry>
+    </collision>
+    <visual>
+      <origin xyz="0 0 0.0" rpy="0 0 0"/>
+      <geometry>
+         <mesh filename="package://robot_description/new_meshes/grinder.stl" scale="0.001 0.001 0.001"/>
+      </geometry>
+      <material name="white"/>
+    </visual>
+    <inertial>
+      <origin xyz="0 0 0.0" rpy="0 0 0"/>
+      <mass value="0.050"/>
+      <inertia ixx="1.0" ixy="0.0" ixz="0.0" iyy="1.0" iyz="0.0" izz="1.0"/>
+    </inertial>
+  </link>
    </robot>

Commit message: Adding rotation part of the topic command, change limit of joints

File: robot_description/model/robot.urdf.xacro (robot description, xacro)
@@ -69,5 +69,5 @@
     <origin xyz="0 0.0 0.044" rpy="0 0 0"/>
     <axis xyz="0 0 1"/>
-    <limit velocity="4.8" effort="1" lower="-1.56" upper="1.56" />
+    <limit velocity="4.8" effort="1" lower="-3.14" upper="3.14" />
   </joint>
   <!-- link_2 -->
@@ -98,5 +98,5 @@
     <origin xyz="0 0.0 0.058" rpy="0 0 0"/>
     <axis xyz="0 1 0"/>
-    <limit velocity="4.8" effort="1" lower="-1.56" upper="1.56" />
+    <limit velocity="4.8" effort="1" lower="-2.2" upper="2.2" />
   </joint>
   <!-- link_3 -->
@@ -127,5 +127,5 @@
     <origin xyz="0 0.0 0.12" rpy="0 0 0"/>
     <axis xyz="0 1 0"/>
-    <limit velocity="4.8" effort="1" lower="-1.56" upper="1.56" />
+    <limit velocity="4.8" effort="1" lower="-2.1" upper="2.1" />
   </joint>
   <!-- link_4 -->
@@ -156,5 +156,5 @@
     <origin xyz="0 0 0.12" rpy="0 0 0"/>
     <axis xyz="0 1 0"/>
-    <limit effort="4.8" lower="-1.56" upper="1.56" velocity="10"/>
+    <limit effort="4.8" lower="-2.1" upper="2.1" velocity="10"/>
   </joint>
   <!-- EndEffector -->
