Commit message: Adding taking account of the gripper

File: robot_description/model/robot_with_gripper.urdf.xacro (robot description, xacro)
@@ -4,12 +4,12 @@
  <xacro:include filename="$(find robot_description)/model/materials.xacro" />
   <!-- World -->
-  <link name="world_link">
-  </link>
+  <!--<link name="world_link">
+  </link>-->
   <!-- World fixed joint-->
-  <joint name="world_fixed_joint" type="fixed">
+  <!--<joint name="world_fixed_joint" type="fixed">
     <origin xyz="0 0 0" rpy="0 0 0"/>
     <parent link="world_link"/>
     <child link="base_link"/>
-  </joint>
+  </joint>-->
   <link name="base_link">
     <inertial>
@@ -129,5 +129,5 @@
     <origin xyz="0 0.0 0.044" rpy="0 0 0"/>
     <axis xyz="0 0 1"/>
-    <limit velocity="4.8" effort="1" lower="-3.14" upper="3.14" />
+    <limit velocity="0.8" effort="1" lower="-3.14" upper="3.14" />
   </joint>
   <!-- link_2 -->
@@ -245,5 +245,5 @@
     <origin xyz="0 -0.046 0.069" rpy="0 0 0"/>
     <axis xyz="0 1 0"/>
-    <limit velocity="4.8" effort="1" lower="-0.010" upper="0.019" />
+    <limit velocity="4.8" effort="1" lower="0.010" upper="0.019" />
   </joint>
   <!-- GripperLeft -->

Commit message: Solving pb of gripper mvmt in rviz

File: robot_description/model/robot_with_gripper.urdf.xacro (robot description, xacro)
@@ -243,7 +243,8 @@
     <parent link="link_5"/>
     <child link="link_gripper_left"/>
-    <origin xyz="0 -0.046 0.069" rpy="0 0 0"/>
-    <axis xyz="0 1 0"/>
-    <limit velocity="4.8" effort="1" lower="0.010" upper="0.019" />
+    <origin xyz="0 -0.0245 0.069" rpy="0 0 0"/>
+    <axis xyz="0 1 0"/>
+    <!--<limit velocity="4.8" effort="1" lower="-0.0245" upper="-0.0455" />-->
+    <limit velocity="4.8" effort="1" lower="0.0" upper="-0.021" />
   </joint>
   <!-- GripperLeft -->
@@ -272,7 +273,8 @@
     <parent link="link_5"/>
     <child link="link_gripper_right"/>
-    <origin xyz="0 0.046 0.069" rpy="0 0 0"/>
-    <axis xyz="0 1 0"/>
-    <limit velocity="4.8" effort="1" lower="-0.010" upper="0.019" />
+    <origin xyz="0 0.0245 0.069" rpy="0 0 0"/>
+    <axis xyz="0 1 0"/>
+    <!--<limit velocity="4.8" effort="1" lower="0.0245" upper="0.0455" />-->
+    <limit velocity="4.8" effort="1" lower="0.0" upper="0.021" />
     <mimic joint="joint5" multiplier="-1" />
   </joint>

Commit message: Changing wheel position and link1 position also in the urdf file

File: robot_description/model/robot_with_gripper.urdf.xacro (robot description, xacro)
@@ -38,5 +38,5 @@
     <parent link="base_link"/>
     <child link="wheel_left_link"/>
-    <origin xyz="0.06 -0.073 0.055" rpy="0 0 0"/>
+    <origin xyz="-0.06 -0.073 0.055" rpy="0 0 0"/>
     <axis xyz="0 1 0"/>
   </joint>
@@ -68,5 +68,5 @@
     <parent link="base_link"/>
     <child link="wheel_right_link"/>
-    <origin xyz="0.06 0.073 0.055" rpy="0 0 0"/>
+    <origin xyz="-0.06 0.073 0.055" rpy="0 0 0"/>
     <axis xyz="0 1 0"/>
   </joint>
